Commit message: Added IMU (inertial measurement unit). Added class robot

File: robot_tppo/urdf/lidar.urdf.xacro (robot description, xacro)
@@ -23,10 +23,10 @@
       </geometry>
     </collision>
-    <visual name='scan_link_visual'>
+    <!--visual name='scan_link_visual'>
       <origin xyz="0 0 0" rpy="0 0 0"/>
       <geometry>
-        <!--mesh filename = "lidar.dae"/-->
+        <mesh filename = "lidar.dae"/>
       </geometry>
-    </visual>
+    </visual-->
 </link>
   <gazebo reference="scan_link">

File: robot_tppo/urdf/robot.urdf.xacro (robot description, xacro)
@@ -4,4 +4,5 @@
     <xacro:include filename="camera.urdf.xacro"/>
     <xacro:include filename="lidar.urdf.xacro"/>
+    <xacro:include filename="inertial_measuring_unit.urdf.xacro"/>
     <ros2_control name="my_robot_hardware" type="system">
         <hardware>
